File: Eagle/Caja_Navidad.brd (EAGLE design)
At the start: 85.1 x 82.2 mm, 24 parts, among them IC1 PIC16F877P

Commit message: add Eagle Files v2
Parts:
- R_LEDS4: value 330 -> (none)
- renumbered POWER_STEP_MOTOR to ALIMENTACION_STEP_MOTOR
Changed lines of the file:
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@@
 <attribute name="VALUE" x="73.66" y="72.644" size="1.27" layer="27" ratio="10" rot="R180"/>
 </element>
-<element name="POWER_STEP_MOTOR" library="jumper" library_urn="urn:adsk.eagle:library:252" package="JP1" package3d_urn="urn:adsk.eagle:package:15455/1" value="" x="76.2" y="68.58" smashed="yes" rot="R270">
+<element name="ALIMENTACION_STEP_MOTOR" library="jumper" library_urn="urn:adsk.eagle:library:252" package="JP1" package3d_urn="urn:adsk.eagle:package:15455/1" value="" x="76.2" y="68.58" smashed="yes" rot="R270">
 <attribute name="NAME" x="73.66" y="70.231" size="1.27" layer="25" ratio="10"/>
 <attribute name="POPULARITY" value="61" x="33.02" y="-33.02" size="1.778" layer="27" rot="R270" display="off"/>
@@
 <attribute name="VALUE" x="97.3074" y="38.4556" size="0.9906" layer="27" ratio="10" rot="R270"/>
 </element>
-<element name="R_LEDS4" library="rcl" library_urn="urn:adsk.eagle:library:334" package="0204/7" package3d_urn="urn:adsk.eagle:package:23498/2" value="330" x="95.25" y="36.83" smashed="yes" rot="R270">
+<element name="R_LEDS4" library="rcl" library_urn="urn:adsk.eagle:library:334" package="0204/7" package3d_urn="urn:adsk.eagle:package:23498/2" value="" x="95.25" y="36.83" smashed="yes" rot="R270">
 <attribute name="NAME" x="96.5454" y="39.37" size="0.9906" layer="25" ratio="10" rot="R270"/>
 <attribute name="POPULARITY" value="79" x="95.25" y="36.83" size="1.778" layer="27" rot="R270" display="off"/>
@@
 <contactref element="DISPLAY_LCD" pad="16"/>
 <contactref element="TRIMMER_LCD" pad="3"/>
-<contactref element="POWER_STEP_MOTOR" pad="2"/>
+<contactref element="ALIMENTACION_STEP_MOTOR" pad="2"/>
 <contactref element="BUZZER" pad="-"/>
 <contactref element="DC-IN" pad="2"/>
@@
 <contactref element="DISPLAY_LCD" pad="2"/>
 <contactref element="TRIMMER_LCD" pad="1"/>
-<contactref element="POWER_STEP_MOTOR" pad="1"/>
+<contactref element="ALIMENTACION_STEP_MOTOR" pad="1"/>
 <contactref element="DC-IN" pad="1"/>
 <contactref element="ALIMENTACION_PICKIT" pad="1"/>
